Commit message: [demos] kukabot retail demo tweaks

File: cram_demos/cram_projection_demos/resource/retail/full_store.urdf.xacro (robot description, xacro)
@@ -14,11 +14,8 @@
         <mesh filename="package://refills_models/shelf_models/ShelfSystemH200T7L10W/ShelfSystemH200T7L10W.dae"/>
       </geometry>
-      <material name="green">
-        <color rgba="0.7 0.7 0.7 1.0"/>
-      </material>
-    </visual>
-    <collision>
-      <geometry>
-        <mesh filename="package://refills_models/shelf_models/ShelfSystemH200T7L10W/ShelfSystemH200T7L10W.dae"/>
+    </visual>
+    <collision>
+      <geometry>
+        <mesh filename="package://refills_models/shelf_models/ShelfSystemH200T7L10W/ShelfSystemH200T7L10W.obj"/>
       </geometry>
     </collision>
@@ -34,7 +31,4 @@
         <mesh filename="package://refills_models/shelf_models/ShelfLayer7TilesL10_Bottom/ShelfLayer7TilesL10_Bottom.dae"/>
       </geometry>
-      <material name="green">
-        <color rgba="0.7 0.7 0.7 1.0"/>
-      </material>
     </visual>
     <collision>
@@ -54,7 +48,4 @@
         <mesh filename="package://refills_models/shelf_models/ShelfSeparator/SM_ShelfSeparator.dae"/>
       </geometry>
-      <material name="green">
-        <color rgba="0.7 0.7 0.7 1.0"/>
-      </material>
     </visual>
     <collision>
@@ -74,7 +65,4 @@
         <mesh filename="package://refills_models/shelf_models/ShelfSeparator/SM_ShelfSeparator.dae"/>
       </geometry>
-      <material name="green">
-        <color rgba="0.7 0.7 0.7 1.0"/>
-      </material>
     </visual>
     <collision>
@@ -94,7 +82,4 @@
         <mesh filename="package://refills_models/shelf_models/ShelfSeparator/SM_ShelfSeparator.dae"/>
       </geometry>
-      <material name="green">
-        <color rgba="0.7 0.7 0.7 1.0"/>
-      </material>
     </visual>
     <collision>
@@ -114,7 +99,4 @@
         <mesh filename="package://refills_models/shelf_models/ShelfSeparator/SM_ShelfSeparator.dae"/>
       </geometry>
-      <material name="green">
-        <color rgba="0.7 0.7 0.7 1.0"/>
-      </material>
     </visual>
     <collision>
@@ -134,7 +116,4 @@
         <mesh filename="package://refills_models/shelf_models/ShelfSeparator/SM_ShelfSeparator.dae"/>
       </geometry>
-      <material name="green">
-        <color rgba="0.7 0.7 0.7 1.0"/>
-      </material>
     </visual>
     <collision>
@@ -154,7 +133,4 @@
         <mesh filename="package://refills_models/shelf_models/ShelfSeparator/SM_ShelfSeparator.dae"/>
       </geometry>
-      <material name="green">
-        <color rgba="0.7 0.7 0.7 1.0"/>
-      </material>
     </visual>
     <collision>
@@ -174,7 +150,4 @@
         <mesh filename="package://refills_models/shelf_models/ShelfSeparator/SM_ShelfSeparator.dae"/>
       </geometry>
-      <material name="green">
-        <color rgba="0.7 0.7 0.7 1.0"/>
-      </material>
     </visual>
     <collision>
@@ -194,11 +167,8 @@
         <mesh filename="package://refills_models/shelf_models/ShelfLayer6TilesL10/ShelfLayer6TilesL10.dae"/>
       </geometry>
-      <material name="green">
-        <color rgba="0.7 0.7 0.7 1.0"/>
-      </material>
-    </visual>
-    <collision>
-      <geometry>
-        <mesh filename="package://refills_models/shelf_models/ShelfLayer6TilesL10/ShelfLayer6TilesL10.dae"/>
+    </visual>
+    <collision>
+      <geometry>
+        <mesh filename="package://refills_models/shelf_models/ShelfLayer6TilesL10/ShelfLayer6TilesL10.obj"/>
       </geometry>
     </collision>
@@ -214,7 +184,4 @@
         <mesh filename="package://refills_models/shelf_models/ShelfSeparator/SM_ShelfSeparator.dae"/>
       </geometry>
-      <material name="green">
-        <color rgba="0.7 0.7 0.7 1.0"/>
-      </material>
     </visual>
     <collision>
@@ -234,7 +201,4 @@
         <mesh filename="package://refills_models/shelf_models/ShelfSeparator/SM_ShelfSeparator.dae"/>
       </geometry>
-      <material name="green">
-        <color rgba="0.7 0.7 0.7 1.0"/>
-      </material>
     </visual>
     <collision>
@@ -254,7 +218,4 @@
         <mesh filename="package://refills_models/shelf_models/ShelfSeparator/SM_ShelfSeparator.dae"/>
       </geometry>
-      <material name="green">
-        <color rgba="0.7 0.7 0.7 1.0"/>
-      </material>
     </visual>
     <collision>
@@ -274,7 +235,4 @@
         <mesh filename="package://refills_models/shelf_models/ShelfSeparator/SM_ShelfSeparator.dae"/>
       </geometry>
-      <material name="green">
-        <color rgba="0.7 0.7 0.7 1.0"/>
-      </material>
     </visual>
     <collision>
@@ -294,7 +252,4 @@
         <mesh filename="package://refills_models/shelf_models/ShelfSeparator/SM_ShelfSeparator.dae"/>
       </geometry>
-      <material name="green">
-        <color rgba="0.7 0.7 0.7 1.0"/>
-      </material>
     </visual>
     <collision>
@@ -314,7 +269,4 @@
         <mesh filename="package://refills_models/shelf_models/ShelfSeparator/SM_ShelfSeparator.dae"/>
       </geometry>
-      <material name="green">
-        <color rgba="0.7 0.7 0.7 1.0"/>
-      </material>
     </visual>
     <collision>
@@ -334,7 +286,4 @@
         <mesh filename="package://refills_models/shelf_models/ShelfSeparator/SM_ShelfSeparator.dae"/>
       </geometry>
-      <material name="green">
-        <color rgba="0.7 0.7 0.7 1.0"/>
-      </material>
     </visual>
     <collision>
@@ -354,11 +303,8 @@
         <mesh filename="package://refills_models/shelf_models/ShelfLayer6TilesL10/ShelfLayer6TilesL10.dae"/>
       </geometry>
-      <material name="green">
-        <color rgba="0.7 0.7 0.7 1.0"/>
-      </material>
-    </visual>
-    <collision>
-      <geometry>
-        <mesh filename="package://refills_models/shelf_models/ShelfLayer6TilesL10/ShelfLayer6TilesL10.dae"/>
+    </visual>
+    <collision>
+      <geometry>
+        <mesh filename="package://refills_models/shelf_models/ShelfLayer6TilesL10/ShelfLayer6TilesL10.obj"/>
       </geometry>
     </collision>
@@ -374,7 +320,4 @@
         <mesh filename="package://refills_models/shelf_models/ShelfSeparator/SM_ShelfSeparator.dae"/>
       </geometry>
-      <material name="green">
-        <color rgba="0.7 0.7 0.7 1.0"/>
-      </material>
     </visual>
     <collision>
@@ -394,7 +337,4 @@
         <mesh filename="package://refills_models/shelf_models/ShelfSeparator/SM_ShelfSeparator.dae"/>
       </geometry>
-      <material name="green">
-        <color rgba="0.7 0.7 0.7 1.0"/>
-      </material>
     </visual>
     <collision>
@@ -414,7 +354,4 @@
         <mesh filename="package://refills_models/shelf_models/ShelfSeparator/SM_ShelfSeparator.dae"/>
       </geometry>
-      <material name="green">
-        <color rgba="0.7 0.7 0.7 1.0"/>
-      </material>
     </visual>
     <collision>
@@ -434,7 +371,4 @@
         <mesh filename="package://refills_models/shelf_models/ShelfSeparator/SM_ShelfSeparator.dae"/>
       </geometry>
-      <material name="green">
-        <color rgba="0.7 0.7 0.7 1.0"/>
-      </material>
     </visual>
     <collision>
@@ -454,7 +388,4 @@
         <mesh filename="package://refills_models/shelf_models/ShelfSeparator/SM_ShelfSeparator.dae"/>
       </geometry>
-      <material name="green">
-        <color rgba="0.7 0.7 0.7 1.0"/>
-      </material>
     </visual>
     <collision>
@@ -474,11 +405,8 @@
         <mesh filename="package://refills_models/shelf_models/ShelfLayer6TilesL10/ShelfLayer6TilesL10.dae"/>
       </geometry>
-      <material name="green">
-        <color rgba="0.7 0.7 0.7 1.0"/>
-      </material>
-    </visual>
-    <collision>
-      <geometry>
-        <mesh filename="package://refills_models/shelf_models/ShelfLayer6TilesL10/ShelfLayer6TilesL10.dae"/>
+    </visual>
+    <collision>
+      <geometry>
+        <mesh filename="package://refills_models/shelf_models/ShelfLayer6TilesL10/ShelfLayer6TilesL10.obj"/>
       </geometry>
     </collision>
@@ -494,7 +422,4 @@
         <mesh filename="package://refills_models/shelf_models/ShelfSeparator/SM_ShelfSeparator.dae"/>
       </geometry>
-      <material name="green">
-        <color rgba="0.7 0.7 0.7 1.0"/>
-      </material>
     </visual>
     <collision>
@@ -514,7 +439,4 @@
         <mesh filename="package://refills_models/shelf_models/ShelfSeparator/SM_ShelfSeparator.dae"/>
       </geometry>
-      <material name="green">
-        <color rgba="0.7 0.7 0.7 1.0"/>
-      </material>
     </visual>
     <collision>
@@ -534,7 +456,4 @@
         <mesh filename="package://refills_models/shelf_models/ShelfSeparator/SM_ShelfSeparator.dae"/>
       </geometry>
-      <material name="green">
-        <color rgba="0.7 0.7 0.7 1.0"/>
-      </material>
     </visual>
     <collision>
@@ -554,7 +473,4 @@
         <mesh filename="package://refills_models/shelf_models/ShelfSeparator/SM_ShelfSeparator.dae"/>
       </geometry>
-      <material name="green">
-        <color rgba="0.7 0.7 0.7 1.0"/>
-      </material>
     </visual>
     <collision>
@@ -574,7 +490,4 @@
         <mesh filename="package://refills_models/shelf_models/ShelfSeparator/SM_ShelfSeparator.dae"/>
       </geometry>
-      <material name="green">
-        <color rgba="0.7 0.7 0.7 1.0"/>
-      </material>
     </visual>
     <collision>
@@ -594,7 +507,4 @@
         <mesh filename="package://refills_models/shelf_models/ShelfSystemH180T510W/SM_ShelfSystemH180T5L10W.dae"/>
       </geometry>
-      <material name="green">
-        <color rgba="0.7 0.7 0.7 1.0"/>
-      </material>
     </visual>
     <collision>
@@ -614,7 +524,4 @@
         <mesh filename="package://refills_models/shelf_models/ShelfLayer5TilesL10_Bottom/ShelfLayer5TilesL10_Bottom.dae"/>
       </geometry>
-      <material name="green">
-        <color rgba="0.7 0.7 0.7 1.0"/>
-      </material>
     </visual>
     <collision>
@@ -634,7 +541,4 @@
         <mesh filename="package://refills_models/shelf_models/ShelfSeparator/SM_ShelfSeparator.dae"/>
       </geometry>
-      <material name="green">
-        <color rgba="0.7 0.7 0.7 1.0"/>
-      </material>
     </visual>
     <collision>
@@ -654,7 +558,4 @@
         <mesh filename="package://refills_models/shelf_models/ShelfSeparator/SM_ShelfSeparator.dae"/>
       </geometry>
-      <material name="green">
-        <color rgba="0.7 0.7 0.7 1.0"/>
-      </material>
     </visual>
     <collision>
@@ -674,7 +575,4 @@
         <mesh filename="package://refills_models/shelf_models/ShelfSeparator/SM_ShelfSeparator.dae"/>
       </geometry>
-      <material name="green">
-        <color rgba="0.7 0.7 0.7 1.0"/>
-      </material>
     </visual>
     <collision>
@@ -694,7 +592,4 @@
         <mesh filename="package://refills_models/shelf_models/ShelfSeparator/SM_ShelfSeparator.dae"/>
       </geometry>
-      <material name="green">
-        <color rgba="0.7 0.7 0.7 1.0"/>
-      </material>
     </visual>
     <collision>
@@ -714,7 +609,4 @@
         <mesh filename="package://refills_models/shelf_models/ShelfSeparator/SM_ShelfSeparator.dae"/>
       </geometry>
-      <material name="green">
-        <color rgba="0.7 0.7 0.7 1.0"/>
-      </material>
     </visual>
     <collision>
@@ -734,11 +626,8 @@
         <mesh filename="package://refills_models/shelf_models/ShelfLayer4TilesL10/ShelfLayer4TilesL10.dae"/>
       </geometry>
-      <material name="green">
-        <color rgba="0.7 0.7 0.7 1.0"/>
-      </material>
-    </visual>
-    <collision>
-      <geometry>
-        <mesh filename="package://refills_models/shelf_models/ShelfLayer4TilesL10/ShelfLayer4TilesL10.dae"/>
+    </visual>
+    <collision>
+      <geometry>
+        <mesh filename="package://refills_models/shelf_models/ShelfLayer4TilesL10/ShelfLayer4TilesL10.obj"/>
       </geometry>
     </collision>
@@ -754,7 +643,4 @@
         <mesh filename="package://refills_models/shelf_models/ShelfSeparator/SM_ShelfSeparator.dae"/>
       </geometry>
-      <material name="green">
-        <color rgba="0.7 0.7 0.7 1.0"/>
-      </material>
     </visual>
     <collision>
@@ -774,7 +660,4 @@
         <mesh filename="package://refills_models/shelf_models/ShelfSeparator/SM_ShelfSeparator.dae"/>
       </geometry>
-      <material name="green">
-        <color rgba="0.7 0.7 0.7 1.0"/>
-      </material>
     </visual>
     <collision>
@@ -794,7 +677,4 @@
         <mesh filename="package://refills_models/shelf_models/ShelfSeparator/SM_ShelfSeparator.dae"/>
       </geometry>
-      <material name="green">
-        <color rgba="0.7 0.7 0.7 1.0"/>
-      </material>
     </visual>
     <collision>
@@ -814,7 +694,4 @@
         <mesh filename="package://refills_models/shelf_models/ShelfSeparator/SM_ShelfSeparator.dae"/>
       </geometry>
-      <material name="green">
-        <color rgba="0.7 0.7 0.7 1.0"/>
-      </material>
     </visual>
     <collision>
@@ -834,7 +711,4 @@
         <mesh filename="package://refills_models/shelf_models/ShelfSeparator/SM_ShelfSeparator.dae"/>
       </geometry>
-      <material name="green">
-        <color rgba="0.7 0.7 0.7 1.0"/>
-      </material>
     </visual>
     <collision>
@@ -854,11 +728,8 @@
         <mesh filename="package://refills_models/shelf_models/ShelfLayer4TilesL10/ShelfLayer4TilesL10.dae"/>
       </geometry>
-      <material name="green">
-        <color rgba="0.7 0.7 0.7 1.0"/>
-      </material>
-    </visual>
-    <collision>
-      <geometry>
-        <mesh filename="package://refills_models/shelf_models/ShelfLayer4TilesL10/ShelfLayer4TilesL10.dae"/>
+    </visual>
+    <collision>
+      <geometry>
+        <mesh filename="package://refills_models/shelf_models/ShelfLayer4TilesL10/ShelfLayer4TilesL10.obj"/>
       </geometry>
     </collision>
@@ -874,7 +745,4 @@
         <mesh filename="package://refills_models/shelf_models/ShelfSeparator/SM_ShelfSeparator.dae"/>
       </geometry>
-      <material name="green">
-        <color rgba="0.7 0.7 0.7 1.0"/>
-      </material>
     </visual>
     <collision>
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
Commit message: [proj-demos] more tweaks for kukabot demo

File: cram_demos/cram_projection_demos/resource/retail/full_store.urdf.xacro (robot description, xacro)
@@ -3,4 +3,10 @@
        xmlns:xacro="http://ros.org/wiki/xacro">
   <xacro:include filename="$(find cram_projection_demos)/resource/retail/store_walls.urdf.xacro"/>
+  <link name="world"/>
+  <joint name="world_to_root" type="fixed">
+    <origin xyz="0 0 0" rpy="0 0 0"/>
+    <parent link="world"/>
+    <child link="store_root"/>
+  </joint>
   <link name="store_root"/>
   <joint name="DMShelfW100_FVHEZLXN" type="fixed">

File: cram_demos/cram_projection_demos/resource/retail/store_walls.urdf.xacro (robot description, xacro)
@@ -8,4 +8,7 @@
           <box size="${size}"/>
         </geometry>
+        <material name="green">
+          <color rgba="0.5 0.5 0.5 1.0"/>
+        </material>
       </visual>
       <collision>
