Commit message: [proj-demos] centralized STORAGE environment and removed highest and second lowest tiers:
the robot's didn't like them :)

File: cram_demos/cram_projection_demos/resource/retail/storage.urdf.xacro (robot description, xacro)
@@ -6,5 +6,5 @@
     <color rgba="0.8 0.8 0.8 1"/>
   </material>
-  <link name="shelf_origin"/>
+  <link name="storage_origin"/>
   <!-- WALLS -->
   <xacro:macro name="wall" params="parent name size *origin">
@@ -29,20 +29,20 @@
   <xacro:property name="wall_thickness" value="0.2" />
   <xacro:property name="wall_height" value="2.4" />
-  <xacro:property name="room_link" value="shelf_origin" />
+  <xacro:property name="room_link" value="storage_origin" />
   <wall parent="${room_link}" name="back_wall"
         size="6.0 ${wall_thickness} ${wall_height}">
-    <origin xyz="-2.0 -2.0 ${wall_height/2}" rpy="0 0 0"/>
+    <origin xyz="0.0 -2.0 ${wall_height/2}" rpy="0 0 0"/>
   </wall>
   <wall parent="${room_link}" name="left_wall"
         size="${wall_thickness} 4.0 ${wall_height}">
-    <origin xyz="1.0 0.0 ${wall_height/2}" rpy="0 0 0"/>
+    <origin xyz="3.0 0.0 ${wall_height/2}" rpy="0 0 0"/>
   </wall>
   <wall parent="${room_link}" name="front_wall"
         size="6.0 ${wall_thickness} ${wall_height}">
-    <origin xyz="-2.0 2.0 ${wall_height/2}" rpy="0 0 0"/>
+    <origin xyz="0.0 2.0 ${wall_height/2}" rpy="0 0 0"/>
   </wall>
   <wall parent="${room_link}" name="right_wall"
         size="${wall_thickness} 4.0 ${wall_height}">
-    <origin xyz="-5.0 0.0 ${wall_height/2}" rpy="0 0 0"/>
+    <origin xyz="-3.0 0.0 ${wall_height/2}" rpy="0 0 0"/>
   </wall>
   <!-- SHELF -->
@@ -122,5 +122,35 @@
     </collision>
   </link>
-  <link name="board1">
+  <!-- <link name="board1"> -->
+  <!--   <visual> -->
+  <!--     <material name="grey"/> -->
+  <!--     <origin xyz="0 0.25 0"/> -->
+  <!--     <geometry> -->
+  <!--       <box size="2 0.5 0.05"/> -->
+  <!--     </geometry> -->
+  <!--   </visual> -->
+  <!--   <collision> -->
+  <!--     <origin xyz="0 0.25 0"/> -->
+  <!--     <geometry> -->
+  <!--       <box size="2 0.5 0.05"/> -->
+  <!--     </geometry> -->
+  <!--   </collision> -->
+  <!-- </link> -->
+  <link name="bar2">
+    <visual>
+      <material name="grey"/>
+      <origin xyz="-1 0 0"/>
+      <geometry>
+        <box size="2 0.1 0.1"/>
+      </geometry>
+    </visual>
+    <collision>
+      <origin xyz="-1 0 0"/>
+      <geometry>
+        <box size="2 0.1 0.1"/>
+      </geometry>
+    </collision>
+  </link>
+  <link name="board2">
     <visual>
       <material name="grey"/>
@@ -137,34 +167,4 @@
     </collision>
   </link>
-  <link name="bar2">
-    <visual>
-      <material name="grey"/>
-      <origin xyz="-1 0 0"/>
-      <geometry>
-        <box size="2 0.1 0.1"/>
-      </geometry>
-    </visual>
-    <collision>
-      <origin xyz="-1 0 0"/>
-      <geometry>
-        <box size="2 0.1 0.1"/>
-      </geometry>
-    </collision>
-  </link>
-  <link name="board2">
-    <visual>
-      <material name="grey"/>
-      <origin xyz="0 0.25 0"/>
-      <geometry>
-        <box size="2 0.5 0.05"/>
-      </geometry>
-    </visual>
-    <collision>
-      <origin xyz="0 0.25 0"/>
-      <geometry>
-        <box size="2 0.5 0.05"/>
-      </geometry>
-    </collision>
-  </link>
   <link name="bar3">
     <visual>
@@ -182,19 +182,19 @@
     </collision>
   </link>
-  <link name="board3">
-    <visual>
-      <material name="grey"/>
-      <origin xyz="0 0.25 0"/>
-      <geometry>
-        <box size="2 0.5 0.05"/>
-      </geometry>
-    </visual>
-    <collision>
-      <origin xyz="0 0.25 0"/>
-      <geometry>
-        <box size="2 0.5 0.05"/>
-      </geometry>
-    </collision>
-  </link>
+  <!-- <link name="board3"> -->
+  <!--   <visual> -->
+  <!--     <material name="grey"/> -->
+  <!--     <origin xyz="0 0.25 0"/> -->
+  <!--     <geometry> -->
+  <!--       <box size="2 0.5 0.05"/> -->
+  <!--     </geometry> -->
+  <!--   </visual> -->
+  <!--   <collision> -->
+  <!--     <origin xyz="0 0.25 0"/> -->
+  <!--     <geometry> -->
+  <!--       <box size="2 0.5 0.05"/> -->
+  <!--     </geometry> -->
+  <!--   </collision> -->
+  <!-- </link> -->
   <joint name="board0_to_bar0" type="fixed">
     <parent link="bar0"/>
@@ -202,9 +202,9 @@
     <origin xyz="-1 0 0"/>
   </joint>
-  <joint name="board1_to_bar1" type="fixed">
-    <parent link="bar1"/>
-    <child link="board1"/>
-    <origin xyz="-1 0 0"/>
-  </joint>
+  <!-- <joint name="board1_to_bar1" type="fixed"> -->
+  <!--   <parent link="bar1"/> -->
+  <!--   <child link="board1"/> -->
+  <!--   <origin xyz="-1 0 0"/> -->
+  <!-- </joint> -->
   <joint name="board2_to_bar2" type="fixed">
     <parent link="bar2"/>
@@ -212,9 +212,9 @@
     <origin xyz="-1 0 0"/>
   </joint>
-  <joint name="board3_to_bar3" type="fixed">
-    <parent link="bar3"/>
-    <child link="board3"/>
-    <origin xyz="-1 0 0"/>
-  </joint>
+  <!-- <joint name="board3_to_bar3" type="fixed"> -->
+  <!--   <parent link="bar3"/> -->
+  <!--   <child link="board3"/> -->
+  <!--   <origin xyz="-1 0 0"/> -->
+  <!-- </joint> -->
   <joint name="bar3_to_left_leg" type="fixed">
     <parent link="left_leg"/>
@@ -242,8 +242,8 @@
     <origin xyz="-2 0 0"/>
   </joint>
-  <joint name="left_leg_to_shelf_origin" type="fixed">
-    <parent link="shelf_origin"/>
+  <joint name="left_leg_to_storage_origin" type="fixed">
+    <parent link="storage_origin"/>
     <child link="left_leg"/>
-    <origin xyz="0 -1.5 0"/>
+    <origin xyz="2.0 -0.7 0" rpy="0 0 0.5"/>
   </joint>
   <!-- TABLE -->
@@ -317,7 +317,7 @@
   </link>
   <joint name="origin_to_left_front_leg" type="fixed">
-    <parent link="shelf_origin"/>
+    <parent link="storage_origin"/>
     <child link="left_front_leg"/>
-    <origin xyz="-4 0 0"/>
+    <origin xyz="-2 0 0"/>
   </joint>
   <joint name="left_front_to_back" type="fixed">
